File: ESC_G431-4in1.kicad_pcb (KiCad board)
At the start: 4 copper layers, 46 x 55.5 mm, 222 parts, among them J1 Conn_01x02, J10 Conn_01x03, J11 Conn_01x03, J2 Conn_01x10, J3 Conn_01x04, J4 Conn_01x04, J5 Conn_01x04, J6 Conn_01x03, J7 Conn_01x04, J8 Conn_01x03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

Commit message: ESC 3d model correction and logo
Parts:
- added G***: LOGO, footprints:ckflight_logo, F.Cu at (139.5, 88.0)
Other:
- board text added: "+"
- board text added: "-"
- board text added: "8S"
- board text added: "CKFLIGHT"
